File: 04_Hardware/PCBs/SEBoard/NFC_PN7160.kicad_sch (KiCad schematic)
At the start: 47 parts, among them J7 636101112001, U12 PN7160B1HN_C100E, Y2 ABM8-27.120MHZ-10-D1G-T

Commit message: feat: Updated schematic layout and moved new components to Layout
Parts:
- AE2: footprint SEBoard:L000641-01 -> 000MCLib:L000641-01; symbol SEBoard:L000641-01 -> 000MCLib:L000641-01
- C119, C63: footprint SEBoard:CAPC1608X80N -> 000MCLib:CAPC1608X80N; symbol SEBoard:C1608C0G1H102F080AA -> 000MCLib:C1608C0G1H102F080AA
- C121, C65: footprint SEBoard:CAPC1608X87N -> 000MCLib:CAPC1608X87N; symbol SEBoard:C0603C751F5GACTU -> 000MCLib:C0603C751F5GACTU
- C123, C126, C57, C59: footprint SEBoard:CAP_CL10_SAM -> 000MCLib:CAP_CL10_SAM; symbol SEBoard:06035A680FAT2A -> 000MCLib:06035A680FAT2A
- C125, C61: footprint SEBoard:CAP_CL10_SAM -> 000MCLib:CAP_CL10_SAM; symbol SEBoard:06035A560FAT2A -> 000MCLib:06035A560FAT2A
- C128, C55: footprint SEBoard:CAP_CL10_SAM -> 000MCLib:CAP_CL10_SAM; symbol SEBoard:CL10C390FB81PNC -> 000MCLib:CL10C390FB81PNC
- C130, C53: footprint SEBoard:CAPC1005X55N -> 000MCLib:CAPC1005X55N; symbol SEBoard:GRM1555C1H100JA01D -> 000MCLib:GRM1555C1H100JA01D
- C132, C49: footprint SEBoard:CAPC1005X55N -> 000MCLib:CAPC1005X55N; symbol SEBoard:GRM155R71A104KA01D -> 000MCLib:GRM155R71A104KA01D
- C133, C45: footprint SEBoard:CAPC1608X90N -> 000MCLib:CAPC1608X90N; symbol SEBoard:LMK107BJ475KA-T -> 000MCLib:LMK107BJ475KA-T
- C134: footprint SEBoard:CAPC1005X55N -> 000MCLib:CAPC1005X55N; symbol SEBoard:GRM155R61H105KE05D -> 000MCLib:GRM155R61H105KE05D
- C140, C48, C50, C51: footprint SEBoard:CAPC1005X55N -> 000MCLib:CAPC1005X55N; symbol SEBoard:GRT155R61A225KE01D -> 000MCLib:GRT155R61A225KE01D
- J7: footprint SEBoard:COAX2_636101112001_WRE -> 000MCLib:COAX2_636101112001_WRE; symbol SEBoard:636101112001 -> 000MCLib:636101112001
- L14, L4: footprint SEBoard:LQW18CNR16J00D -> 000MCLib:LQW18CNR16J00D; symbol SEBoard:LQW18CNR16J00D -> 000MCLib:LQW18CNR16J00D
- R136, R72: footprint SEBoard:ERJ3EKF1000V -> 000MCLib:ERJ3EKF1000V; symbol SEBoard:ERJ-3GEYJ222V -> 000MCLib:ERJ-3GEYJ222V
- R139, R140, R141, R142, R144, R70: footprint SEBoard:RC0402N_YAG -> 000MCLib:RC0402N_YAG; symbol SEBoard:RC0402JR-070RL -> 000MCLib:RC0402JR-070RL
- R146, R154: footprint SEBoard:RESC2012X50N -> 000MCLib:RESC2012X50N; symbol SEBoard:CRCW08050000Z0EA -> 000MCLib:CRCW08050000Z0EA
- R151, R68: footprint SEBoard:RESC2012X50N -> 000MCLib:RESC2012X50N; symbol SEBoard:CRCW08052R70FKEA -> 000MCLib:CRCW08052R70FKEA
- R153: footprint SEBoard:RC0402N_YAG -> 000MCLib:RC0402N_YAG; symbol SEBoard:RC0402JR-0710KL -> 000MCLib:RC0402JR-0710KL
- TP57, TP58, TP59, TP60, TP61: symbol SEBoard:TestPoint -> 000MCLib:TestPoint
- U12: footprint SEBoard:QFN50P600X600X100-41N-D -> 000MCLib:QFN50P600X600X100-41N-D; symbol SEBoard:PN7160B1HN_C100E -> 000MCLib:PN7160B1HN_C100E
- Y2: footprint SEBoard:ABM810000MHZ12D2W -> 000MCLib:ABM810000MHZ12D2W; symbol SEBoard:ABM8-27.120MHZ-10-D1G-T -> 000MCLib:ABM8-27.120MHZ-10-D1G-T
