File: 04_Hardware/PCBs/SEBoard/NFC_PN7220.kicad_sch (KiCad schematic)
At the start: 77 parts, among them IC1 PN7220, J7 BM02B-ACHSS-GAN-TF, Q11 BC847C,215, Q12 BC847C,215, Y1 27.120MHz

Commit message: feat: Updated schematic layout and moved new components to Layout
Parts:
- C112, C60, C64: footprint SEBoard:CAPC1005X55N -> 000MCLib:CAPC1005X55N; symbol SEBoard:GRM1555C1H101JA01J -> 000MCLib:GRM1555C1H101JA01J
- C113, C122, C144: footprint SEBoard:CAPC1005X55N -> 000MCLib:CAPC1005X55N; symbol SEBoard:GRM155R71A104KA01D -> 000MCLib:GRM155R71A104KA01D
- C120, C124, C136, C58: footprint SEBoard:CAPC1005X55N -> 000MCLib:CAPC1005X55N; symbol SEBoard:GRM155R61A224JE19D -> 000MCLib:GRM155R61A224JE19D
- C127, C129: footprint SEBoard:CAPC1005X55N -> 000MCLib:CAPC1005X55N; symbol SEBoard:GRM1555C1H100JA01D -> 000MCLib:GRM1555C1H100JA01D
- C131, C137: footprint SEBoard:CAPC1608X80N -> 000MCLib:CAPC1608X80N; symbol SEBoard:C1608C0G1H102F080AA -> 000MCLib:C1608C0G1H102F080AA
- C138, C139: footprint SEBoard:CAPC1608X87N -> 000MCLib:CAPC1608X87N; symbol SEBoard:C0603C751F5GACTU -> 000MCLib:C0603C751F5GACTU
- C45, C48: footprint SEBoard:CAP_CL10_SAM -> 000MCLib:CAP_CL10_SAM; symbol SEBoard:06035A470FAT2A -> 000MCLib:06035A470FAT2A
- C46, C52, C54, C62, C67: footprint SEBoard:CAPC1608X90N -> 000MCLib:CAPC1608X90N; symbol SEBoard:LMK107BJ475KA-T -> 000MCLib:LMK107BJ475KA-T
- C47: footprint SEBoard:CAPC1005X55N -> 000MCLib:CAPC1005X55N; symbol SEBoard:GRM155R61H105KE05D -> 000MCLib:GRM155R61H105KE05D
- C49, C50: footprint SEBoard:CAPC1608X87N -> 000MCLib:CAPC1608X87N; symbol SEBoard:C0603C201F5GACTU -> 000MCLib:C0603C201F5GACTU
- C56: footprint SEBoard:CAPC2012X145N -> 000MCLib:CAPC2012X145N; symbol SEBoard:GRM21BR61E226ME44L -> 000MCLib:GRM21BR61E226ME44L
- IC1: footprint SEBoard:BGA64C50P8X8_450X450X90 -> 000MCLib:BGA64C50P8X8_450X450X90; symbol SEBoard:PN7220 -> 000MCLib:PN7220
- J7: footprint SEBoard:BM02B-ACHSS-GAN-TF -> 000MCLib:BM02B-ACHSS-GAN-TF; symbol SEBoard:BM02B-ACHSS-GAN-TF -> 000MCLib:BM02B-ACHSS-GAN-TF
- L13: footprint SEBoard:LQM2HPN1R0MG0L -> 000MCLib:LQM2HPN1R0MG0L; symbol SEBoard:LQM2HPN1R0MG0L -> 000MCLib:LQM2HPN1R0MG0L
- L15, L16: footprint SEBoard:LQW18CNR16J00D -> 000MCLib:LQW18CNR16J00D; symbol SEBoard:LQW18CNR16J00D -> 000MCLib:LQW18CNR16J00D
- LED6: footprint SEBoard:SMLP11VTT86R -> 000MCLib:SMLP11VTT86R; symbol SEBoard:SML-P11VTT86R -> 000MCLib:SML-P11VTT86R
- LED7: footprint SEBoard:SMLP11VTT86R -> 000MCLib:SMLP11VTT86R; symbol SEBoard:SML-P11YTT86R -> 000MCLib:SML-P11YTT86R
- Q11, Q12: footprint SOT95P230X110-3N -> 000MCLib:SOT95P230X110-3N; symbol SEBoard:BC847C,215 -> 000MCLib:BC847C,215
- R112, R118, R119, R120, R122, R123, R124, R125, R132, R133, R134, R136, R137, R138, R139, R140, R141, R142, R144, R67, R70, R72: footprint SEBoard:RC0402N_YAG -> 000MCLib:RC0402N_YAG; symbol SEBoard:RC0402JR-0710KL -> 000MCLib:RC0402JR-0710KL
- R113, R146: footprint SEBoard:RC0402N_YAG -> 000MCLib:RC0402N_YAG; symbol SEBoard:RC0402JR-071KL -> 000MCLib:RC0402JR-071KL
- R114, R115, R116, R117, R121, R126, R131: footprint SEBoard:RC0402N_YAG -> 000MCLib:RC0402N_YAG; symbol SEBoard:RC0402JR-070RL -> 000MCLib:RC0402JR-070RL
- R127, R128: footprint SEBoard:RC0402N_YAG -> 000MCLib:RC0402N_YAG; symbol SEBoard:RC0402JR-072K2L -> 000MCLib:RC0402JR-072K2L
- R129, R130: footprint SEBoard:RESC2012X70N -> 000MCLib:RESC2012X70N; symbol SEBoard:RCWE080520L0FMEA -> 000MCLib:RCWE080520L0FMEA
- R135, R143: footprint SEBoard:ERJ3EKF1000V -> 000MCLib:ERJ3EKF1000V; symbol SEBoard:ERJ-3GEYJ152V -> 000MCLib:ERJ-3GEYJ152V; Part Number ERJ-3GEYJ222V -> ERJ-3GEYJ152V
- R150: footprint SEBoard:RESC2012X50N -> 000MCLib:RESC2012X50N; symbol SEBoard:CRCW08050000Z0EA -> 000MCLib:CRCW08050000Z0EA
- TP24, TP25: symbol SEBoard:TestPoint -> 000MCLib:TestPoint
- Y1: footprint SEBoard:ABM810000MHZ12D2W -> 000MCLib:ABM810000MHZ12D2W; symbol SEBoard:ABM8-27.120MHZ-10-D1G-T -> 000MCLib:ABM8-27.120MHZ-10-D1G-T
