File: 04_Hardware/PCBs/SEBoard/Power.kicad_sch (KiCad schematic)
At the start: 85 parts, among them IC5 LM74700QDBVRQ1, J1 PJ-059A, J3 53047-0310, J4 67996-100HLF, Q13 AO3400A, U1 SC200EEMNA-E53-UGNDA, U2 RT8279GSP, U3 AP7335-WG-7, U4 AP7343DQ-11W5-7, U8 AP61100Z6-7

Commit message: feat(schematic): add SE250B4 symbol to schematic (unchecked)
Parts:
- removed TP5: LDO15A_1V8, TestPoint:TestPoint_Pad_D1.0mm, symbol SEBoard:TestPoint
- removed U1: SC200EEMNA-E53-UGNDA, SEBoard:SC200E_SC206E, symbol SEBoard:SC200E
- added TP19, TP26: LDO_IOVDD, TestPoint:TestPoint_Pad_D1.0mm, symbol SEBoard:TestPoint
- added U5: SE250B4, 000MCLib:XCVR_SE250B4-NA, symbol 000MCLib:SE250B4
Connections:
- net LDO_IOVDD is gone; now on net LDO15A_1V8: TP6.1
- net BAT_THERM: now also U5.AG5 (BATT_THERM)
- net GND: now also U5.1 (GND_1), U5.10 (GND_10), U5.11 (GND_11), U5.12 (GND_12), U5.13 (GND_13), U5.14 (GND_14), U5.15 (GND_15), U5.16 (GND_16), U5.17 (GND_17), U5.18 (GND_18), U5.19 (GND_19), U5.2 (GND_2), U5.20 (GND_20), U5.21 (GND_21), U5.22 (GND_22), U5.23 (GND_23), U5.24 (GND_24), U5.25 (GND_25), U5.26 (GND_26), U5.27 (GND_27), U5.28 (GND_28), U5.29 (GND_29), U5.3 (GND_3), U5.30 (GND_30), U5.31 (GND_31), U5.32 (GND_32), U5.33 (GND_33), U5.34 (GND_34), U5.35 (GND_35), U5.36 (GND_36), U5.37 (GND_37), U5.38 (GND_38), U5.39 (GND_39), U5.4 (GND_4), U5.40 (GND_40), U5.41 (GND_41), U5.42 (GND_42), U5.43 (GND_43), U5.44 (GND_44), U5.45 (GND_45), U5.46 (GND_46), U5.47 (GND_47), U5.48 (GND_48), U5.49 (GND_49), U5.5 (GND_5), U5.50 (GND_50), U5.51 (GND_51), U5.52 (GND_52), U5.53 (GND_53), U5.54 (GND_54), U5.55 (GND_55), U5.56 (GND_56), U5.57 (GND_57), U5.58 (GND_58), U5.59 (GND_59), U5.6 (GND_6), U5.60 (GND_60), U5.7 (GND_7), U5.8 (GND_8), U5.9 (GND_9), U5.A1 (RKEY), U5.A11 (GND_A11), U5.A15 (GND_A15), U5.A17 (GND_A17), U5.A21 (GND_A21), U5.A23 (GND_A23), U5.A27 (GND_A27), U5.A29 (GND_A29), U5.A31 (GND_A31), U5.A35 (GND_A35), U5.A39 (GND_A39), U5.A43 (GND_A43), U5.A7 (GND_A7), U5.AA47 (GND_AA47), U5.AA5 (GND_AA5), U5.AB45 (GND_AB45), U5.AB51 (GND_AB51), U5.AC50 (GND_AC50), U5.AD7 (GND_AD7), U5.AE5 (GND_AE5), U5.AF3 (GND_AF3), U5.AF45 (GND_AF45), U5.AG2 (GND_AG2), U5.AH1 (GND_AH1), U5.AH51 (GND_AH51), U5.AJ2 (GND_AJ2), U5.AJ47 (GND_AJ47), U5.AJ5 (GND_AJ5), U5.AK3 (GND_AK3), U5.AK45 (GND_AK45), U5.AK51 (GND_AK51), U5.AL2 (GND_AL2), U5.AL47 (GND_AL47), U5.AM1 (GND_AM1), U5.AM45 (GND_AM45), U5.AN2 (GND_AN2), U5.AN50 (GND_AN50), U5.AP1 (GND_AP1), U5.AP51 (GND_AP51), U5.AR2 (GND_AR2), U5.AS1 (GND_AS1), U5.AT2 (GND_AT2), U5.AU1 (GND_AU1), U5.AU45 (GND_AU45), U5.AU51 (GND_AU51), U5.AV47 (GND_AV47), U5.AV50 (GND_AV50), U5.AW49 (GND_AW49), U5.AY1 (GND_AY1), U5.AY11 (GND_AY11), U5.AY17 (GND_AY17), U5.AY19 (GND_AY19), U5.AY29 (GND_AY29), U5.AY33 (GND_AY33), U5.AY37 (GND_AY37), U5.AY39 (GND_AY39), U5.AY41 (GND_AY41), U5.AZ2 (GND_AZ2), U5.B10 (GND_B10), U5.B14 (GND_B14), U5.B16 (GND_B16), U5.B18 (GND_B18), U5.B24 (GND_B24), U5.B26 (GND_B26), U5.B28 (GND_B28), U5.B32 (GND_B32), U5.B34 (GND_B34), U5.B40 (GND_B40), U5.B42 (GND_B42), U5.B8 (GND_B8), U5.BA1 (GND_BA1), U5.BA12 (GND_BA12), U5.BA20 (GND_BA20), U5.BA26 (GND_BA26), U5.BA30 (GND_BA30), U5.BA38 (GND_BA38), U5.BA40 (GND_BA40), U5.BA42 (GND_BA42), U5.BC13 (GND_BC13), U5.BC23 (GND_BC23), U5.BC29 (GND_BC29), U5.BC37 (GND_BC37), U5.BC45 (GND_BC45), U5.BD14 (GND_BD14), U5.BD24 (GND_BD24), U5.BD38 (GND_BD38), U5.BD44 (GND_BD44), U5.BE11 (GND_BE11), U5.BE17 (GND_BE17), U5.BE21 (GND_BE21), U5.BE27 (GND_BE27), U5.BE39 (GND_BE39), U5.BE41 (GND_BE41), U5.BE7 (GND_BE7), U5.C13 (GND_C13), U5.C15 (GND_C15), U5.C33 (GND_C33), U5.C41 (GND_C41), U5.C7 (GND_C7), U5.C9 (GND_C9), U5.E10 (GND_E10), U5.F50 (GND_F50), U5.G1 (GND_G1), U5.H2 (GND_H2), U5.J1 (GND_J1), U5.J51 (GND_J51), U5.M47 (GND_M47), U5.M50 (GND_M50), U5.N49 (GND_N49), U5.N51 (GND_N51), U5.N7 (GND_N7), U5.P47 (GND_P47), U5.P50 (GND_P50), U5.R3 (GND_R3), U5.T45 (GND_T45), U5.U5 (GND_U5), U5.V3 (GND_V3), U5.X1 (GND_X1), U5.Y2 (GND_Y2), U5.Y5 (GND_Y5)
- net LDO15A_1V8: now also U5.AB49 (VREG_L15A_1P8_AB49), U5.AH49 (VREG_L15A_1P8_AH49)
- net LDO17A_3V0: now also U5.AD49 (VREG_L17A_3P0)
- net VBAT: now also U5.AW51 (VPH_PA_AW51), U5.AX50 (VPH_PA_AX50), U5.AY49 (VPH_PA_AY49), U5.AY51 (VPH_PA_AY51), U5.AZ50 (VPH_PA_AZ50), U5.BA51 (VPH_PA_BA51), U5.BC41 (VPH_PA_BC41), U5.BD42 (VPH_PA_BD42), U5.BE47 (VBAT)
- net VDD_2V8: now also U5.AM49 (VREG_L20A_2P96)
- net VPH_PWR: now also U5.BC39 (VPH_PWR_BC39), U5.BC43 (VPH_PWR_BC43), U5.BD40 (VPH_PWR_BD40), U5.BD46 (VPH_PWR_BD46), U5.BE43 (VPH_PWR_BE43), U5.BE45 (VPH_PWR_BE45)
- net at R8.1: now also U5.AK7 (BATT_CONN_VSNS_M)
- net at TP10.1: now also U5.G17 (VCOIN)
- net at R9.1: now also U5.AA2 (CBL_PWR_N)
- net at R7.1: now also U5.AH7 (BATT_CONN_VSNS_P)
- new net: TP26.1, U5.C17 (VREG_S3A_1P352)
- new net: TP19.1, U5.X3 (VREG_S4A_2P04)
- no-connect marks 18 -> 4
Other:
- moved on the sheet: C15, C16, C17, R7, R8, R9, TP10, TP6, TP7, TP8, TP9

Commit message: feat: Updated schematic layout and moved new components to Layout
Parts:
- added unit 9 of U5
- C1: footprint SEBoard:T495X -> 000MCLib:T495X; symbol SEBoard:T495X107M016ATE1007280 -> 000MCLib:T495X107M016ATE1007280
- C10, C17: footprint SEBoard:CAPC1005X55N -> 000MCLib:CAPC1005X55N; symbol SEBoard:GRM1555C1H330JA01D -> 000MCLib:GRM1555C1H330JA01D
- C11, C7: footprint SEBoard:T495D -> 000MCLib:T495D; symbol SEBoard:T495D107K010ATE080 -> 000MCLib:T495D107K010ATE080
- C12, C19, C21, C23, C36, C38, C57, C9: footprint SEBoard:CAPC1005X55N -> 000MCLib:CAPC1005X55N; symbol SEBoard:GRM155R71A104KA01D -> 000MCLib:GRM155R71A104KA01D
- C13: footprint SEBoard:CAPC1005X55N -> 000MCLib:CAPC1005X55N; symbol SEBoard:GRM1555C1H101JA01J -> 000MCLib:GRM1555C1H101JA01J
- C14: footprint SEBoard:CAPC1005X55N -> 000MCLib:CAPC1005X55N; symbol SEBoard:GRM1555C1H102JA01D -> 000MCLib:GRM1555C1H102JA01D
- C15, C61: footprint SEBoard:CAPC1005X55N -> 000MCLib:CAPC1005X55N; symbol SEBoard:GRM158R60J226ME01D -> 000MCLib:GRM158R60J226ME01D
- C16, C18, C20, C22, C35, C37: footprint SEBoard:CAPC1005X55N -> 000MCLib:CAPC1005X55N; symbol SEBoard:GRM155R61H105KE05D -> 000MCLib:GRM155R61H105KE05D
- C2, C3, C66: footprint SEBoard:CAP_UMK325B7475MM-T_TAY -> 000MCLib:CAP_UMK325B7475MM-T_TAY; symbol SEBoard:UMK325BJ475MM-T -> 000MCLib:UMK325BJ475MM-T
- C4: footprint SEBoard:CAPC1005X55N -> 000MCLib:CAPC1005X55N; symbol SEBoard:UMK105B7104KVHF -> 000MCLib:UMK105B7104KVHF
- C43, C44: footprint SEBoard:CAPC1005X55N -> 000MCLib:CAPC1005X55N; symbol SEBoard:GRM155R60J106ME15D -> 000MCLib:GRM155R60J106ME15D
- C5: footprint SEBoard:CAPC1005X55N -> 000MCLib:CAPC1005X55N; symbol SEBoard:GRM155R71H103KA88D -> 000MCLib:GRM155R71H103KA88D
- C59, C8: footprint SEBoard:GRM31x -> 000MCLib:GRM31x; symbol SEBoard:GRM31CR60J476ME19L -> 000MCLib:GRM31CR60J476ME19L
- C6: footprint SEBoard:CAPC1005X55N -> 000MCLib:CAPC1005X55N; symbol SEBoard:GRM1555C1H820JA01D -> 000MCLib:GRM1555C1H820JA01D
- C98: footprint SEBoard:CAPC1005X55N -> 000MCLib:CAPC1005X55N; symbol SEBoard:GRM1555C1H220JA01D -> 000MCLib:GRM1555C1H220JA01D
- D1: footprint SEBoard:SD12CTCT -> 000MCLib:SD12CTCT; symbol SEBoard:SD12C.TCT -> 000MCLib:SD12C.TCT
- D2, D6: footprint SEBoard:SC110501UTG -> 000MCLib:SC110501UTG; symbol SEBoard:SC1105-01UTG -> 000MCLib:SC1105-01UTG
- D3: footprint SEBoard:DIOM7959X250N -> 000MCLib:DIOM7959X250N; symbol SEBoard:B550C-13-F -> 000MCLib:B550C-13-F
- D4: footprint SEBoard:SOD2513X120N -> 000MCLib:SOD2513X120N; symbol SEBoard:B140WS-7 -> 000MCLib:B140WS-7
- D5: footprint SEBoard:SODFL1006X40N -> 000MCLib:SODFL1006X40N; symbol SEBoard:ESD9B5.0ST5G -> 000MCLib:ESD9B5.0ST5G
- IC5: footprint SEBoard:SOT95P280X145-6N -> 000MCLib:SOT95P280X145-6N; symbol SEBoard:LM74700QDBVRQ1 -> 000MCLib:LM74700QDBVRQ1
- J1: footprint SEBoard:PJ059A -> 000MCLib:PJ059A; symbol SEBoard:PJ-059A -> 000MCLib:PJ-059A
- J3: footprint SEBoard:530470310 -> 000MCLib:530470310; symbol SEBoard:53047-0310 -> 000MCLib:53047-0310
- J4: footprint SEBoard:HDRV2W67P254_2X1_254X483X858P -> 000MCLib:HDRV2W67P254_2X1_254X483X858P; symbol SEBoard:67996-100HLF -> 000MCLib:67996-100HLF
- L1: footprint SEBoard:NS10165T220MNA -> 000MCLib:NS10165T220MNA; symbol SEBoard:NS10155T150MNA -> 000MCLib:NS10155T150MNA
- L3: footprint SEBoard:IND_WE-LQS_2512_WRE -> 000MCLib:IND_WE-LQS_2512_WRE; symbol SEBoard:74404024010 -> 000MCLib:74404024010
- Q13: footprint SEBoard:SOT95P280X125-3N -> 000MCLib:SOT95P280X125-3N; symbol SEBoard:AO3400A -> 000MCLib:AO3400A
- R1, R2: footprint SEBoard:RC0402N_YAG -> 000MCLib:RC0402N_YAG; symbol SEBoard:RC0402JR-07100KL -> 000MCLib:RC0402JR-07100KL
- R10, R13, R17, R31: footprint SEBoard:RC0402N_YAG -> 000MCLib:RC0402N_YAG; symbol SEBoard:RC0402JR-0710KL -> 000MCLib:RC0402JR-0710KL
- R11: footprint SEBoard:RC0402N_YAG -> 000MCLib:RC0402N_YAG; symbol SEBoard:RC0402FR-07147KL -> 000MCLib:RC0402FR-07147KL
- R12, R6: footprint SEBoard:RC0402N_YAG -> 000MCLib:RC0402N_YAG; symbol SEBoard:RC0402JR-0747KL -> 000MCLib:RC0402JR-0747KL
- R145, R4, R7, R71, R8, R9: footprint SEBoard:RC0402N_YAG -> 000MCLib:RC0402N_YAG; symbol SEBoard:RC0402JR-070RL -> 000MCLib:RC0402JR-070RL
- R21: footprint SEBoard:RC0402N_YAG -> 000MCLib:RC0402N_YAG; symbol SEBoard:RC0402JR-0710KL -> 000MCLib:RC0402JR-0710KL; now fitted; now in the parts list
- R29: footprint SEBoard:RC0402N_YAG -> 000MCLib:RC0402N_YAG; symbol SEBoard:RC0402FR-0744K2L -> 000MCLib:RC0402FR-0744K2L
- R3: footprint SEBoard:RC0402N_YAG -> 000MCLib:RC0402N_YAG; symbol SEBoard:RC0402JR-0743KL -> 000MCLib:RC0402JR-0743KL
- R30: footprint SEBoard:RC0402N_YAG -> 000MCLib:RC0402N_YAG; symbol SEBoard:RC0402JR-0710KL -> 000MCLib:RC0402JR-0710KL; now not fitted; now left out of the parts list
- R66: footprint SEBoard:RC0402N_YAG -> 000MCLib:RC0402N_YAG; symbol SEBoard:RC0402FR-07200KL -> 000MCLib:RC0402FR-07200KL
- TP1, TP10, TP11, TP12, TP19, TP2, TP26, TP3, TP4, TP6, TP63, TP7, TP8, TP9: symbol SEBoard:TestPoint -> 000MCLib:TestPoint
- U2: footprint SEBoard:SOP8L_EP1_RIT -> 000MCLib:SOP8L_EP1_RIT; symbol SEBoard:RT8279GSP -> 000MCLib:RT8279GSP
- U3: footprint SEBoard:SOT95P285X145-5N -> 000MCLib:SOT95P285X145-5N; symbol SEBoard:AP7335-WG-7 -> 000MCLib:AP7335-WG-7
- U4: footprint SEBoard:SOT95P285X145-5N -> 000MCLib:SOT95P285X145-5N; symbol SEBoard:AP7343DQ-11W5-7 -> 000MCLib:AP7343DQ-11W5-7
- U8: footprint SEBoard:SOT50P162X60-6N -> 000MCLib:SOT50P162X60-6N; symbol SEBoard:AP61100Z6-7 -> 000MCLib:AP61100Z6-7
Connections:
- net GND: now also D3.1 (A); no longer D3.2 (A)
- net at C5.2, L1.1, U2.8 (SW): now also D3.2 (K); no longer D3.1 (K)
Other:
- moved on the sheet: C11, C12, C13, C14, C15, C16, C17, C18, C19, C20, C21, C22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
