File: 04_Hardware/PCBs/SEBoard/Power.kicad_sch (KiCad schematic)
At the start: 86 parts, among them IC5 LM74700QDBVRQ1, J1 PJ-059A, J3 53047-0310, J4 67996-100HLF, Q13 AO3400A, U2 RT8279GSP, U3 AP7335-WG-7, U4 AP7343DQ-11W5-7, U5 SE250B4, U8 AP61100Z6-7

Commit message: Feat: Modified Layout for SE250B4 first version
Parts:
- added C110: 4.7uF 50V, 000MCLib:CAP_UMK325B7475MM-T_TAY, symbol 000MCLib:UMK325BJ475MM-T
Connections:
- net GND: now also C110.2
- net at TP10.1, U5.G17 (VCOIN): now also C110.1
Other:
- moved on the sheet: TP10
