File: 04_Hardware/PCBs/SEBoard/Sensors.kicad_sch (KiCad schematic)
At the start: 18 parts, among them U6 LIS2DH12TR, U7 MMC3630KJ

Commit message: feat: Updated schematic layout and moved new components to Layout
Parts:
- B1: footprint SEBoard:PUI_HD-EMB1104-SM-2 -> 000MCLib:PUI_HD-EMB1104-SM-2; symbol SEBoard:HD-EMB1104-SM-2 -> 000MCLib:HD-EMB1104-SM-2
- C114, C39: footprint SEBoard:CAPC1005X55N -> 000MCLib:CAPC1005X55N; symbol SEBoard:GRM155R71A104KA01D -> 000MCLib:GRM155R71A104KA01D
- C115: footprint SEBoard:CAPC1005X55N -> 000MCLib:CAPC1005X55N; symbol SEBoard:GRM155R60J106ME15D -> 000MCLib:GRM155R60J106ME15D
- C40, C41: footprint SEBoard:CAPC1005X55N -> 000MCLib:CAPC1005X55N; symbol SEBoard:GRM155R61H105KE05D -> 000MCLib:GRM155R61H105KE05D
- C42: footprint SEBoard:CAPC1608X90N -> 000MCLib:CAPC1608X90N; symbol SEBoard:LMK107BJ475KA-T -> 000MCLib:LMK107BJ475KA-T
- D17: footprint SEBoard:SOD2513X120N -> 000MCLib:SOD2513X120N; symbol SEBoard:B140WS-7 -> 000MCLib:B140WS-7
- LED4: footprint SEBoard:SMLP11VTT86R -> 000MCLib:SMLP11VTT86R; symbol SEBoard:SML-P11VTT86R -> 000MCLib:SML-P11VTT86R
- R60: footprint SEBoard:RC0402N_YAG -> 000MCLib:RC0402N_YAG; symbol SEBoard:RC0402JR-0733RL -> 000MCLib:RC0402JR-0733RL
- R61, R62, R65: footprint SEBoard:RC0402N_YAG -> 000MCLib:RC0402N_YAG; symbol SEBoard:RC0402JR-072K2L -> 000MCLib:RC0402JR-072K2L
- R63, R64: footprint SEBoard:RC0402N_YAG -> 000MCLib:RC0402N_YAG; symbol SEBoard:RC0402JR-070RL -> 000MCLib:RC0402JR-070RL
- TP23: symbol SEBoard:TestPoint -> 000MCLib:TestPoint
- U6: footprint SEBoard:LGA-12_STM -> 000MCLib:LGA-12_STM; symbol SEBoard:LIS2DH12TR -> 000MCLib:LIS2DH12TR
- U7: footprint SEBoard:BGA8C40P3X3_120X120X57 -> 000MCLib:BGA8C40P3X3_120X120X57; symbol SEBoard:MMC3630KJ -> 000MCLib:MMC3630KJ
Changed lines of the file:
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@@
 	)
 	(symbol
-		(lib_id "SEBoard:RC0402JR-0733RL")
+		(lib_id "000MCLib:RC0402JR-0733RL")
 		(at 181.61 45.72 0)
 		(unit 1)
@@
 			)
 		)
-		(property "Footprint" "SEBoard:RC0402N_YAG"
+		(property "Footprint" "000MCLib:RC0402N_YAG"
 			(at 175.26 45.72 0)
 			(effects
@@
 	)
 	(symbol
-		(lib_id "SEBoard:GRM155R61H105KE05D")
+		(lib_id "000MCLib:GRM155R61H105KE05D")
 		(at 74.93 63.5 180)
 		(unit 1)
@@
 			)
 		)
-		(property "Footprint" "SEBoard:CAPC1005X55N"
+		(property "Footprint" "000MCLib:CAPC1005X55N"
 			(at 66.04 -32.69 0)
 			(effects
@@
 	)
 	(symbol
-		(lib_id "SEBoard:TestPoint")
+		(lib_id "000MCLib:TestPoint")
 		(at 238.76 45.72 270)
 		(unit 1)
@@
 	)
 	(symbol
-		(lib_id "SEBoard:GRM155R71A104KA01D")
+		(lib_id "000MCLib:GRM155R71A104KA01D")
 		(at 250.19 63.5 270)
 		(unit 1)
@@
 			)
 		)
-		(property "Footprint" "SEBoard:CAPC1005X55N"
+		(property "Footprint" "000MCLib:CAPC1005X55N"
 			(at 154 72.39 0)
 			(effects
@@
 	)
 	(symbol
-		(lib_id "SEBoard:LMK107BJ475KA-T")
+		(lib_id "000MCLib:LMK107BJ475KA-T")
 		(at 55.88 55.88 90)
 		(unit 1)
@@
 			)
 		)
-		(property "Footprint" "SEBoard:CAPC1608X90N"
+		(property "Footprint" "000MCLib:CAPC1608X90N"
 			(at 152.07 46.99 0)
 			(effects
@@
 	)
 	(symbol
-		(lib_id "SEBoard:GRM155R61H105KE05D")
+		(lib_id "000MCLib:GRM155R61H105KE05D")
 		(at 199.39 124.46 270)
 		(unit 1)
@@
 			)
 		)
-		(property "Footprint" "SEBoard:CAPC1005X55N"
+		(property "Footprint" "000MCLib:CAPC1005X55N"
 			(at 103.2 133.35 0)
 			(effects
@@
 	)
 	(symbol
-		(lib_id "SEBoard:RC0402JR-070RL")
+		(lib_id "000MCLib:RC0402JR-070RL")
 		(at 241.3 118.11 180)
 		(unit 1)
@@
 			)
 		)
-		(property "Footprint" "SEBoard:RC0402N_YAG"
+		(property "Footprint" "000MCLib:RC0402N_YAG"
 			(at 247.65 118.11 0)
 			(effects
@@
 	)
 	(symbol
-		(lib_id "SEBoard:RC0402JR-072K2L")
+		(lib_id "000MCLib:RC0402JR-072K2L")
 		(at 116.84 133.35 270)
 		(unit 1)
@@
 			)
 		)
-		(property "Footprint" "SEBoard:RC0402N_YAG"
+		(property "Footprint" "000MCLib:RC0402N_YAG"
 			(at 116.84 127 0)
 			(effects
@@
 	)
 	(symbol
-		(lib_id "SEBoard:GRM155R71A104KA01D")
+		(lib_id "000MCLib:GRM155R71A104KA01D")
 		(at 234.95 63.5 270)
 		(unit 1)
@@
 			)
 		)
-		(property "Footprint" "SEBoard:CAPC1005X55N"
+		(property "Footprint" "000MCLib:CAPC1005X55N"
 			(at 138.76 72.39 0)
 			(effects
@@
 	)
 	(symbol
-		(lib_id "SEBoard:RC0402JR-070RL")
+		(lib_id "000MCLib:RC0402JR-070RL")
 		(at 191.77 118.11 0)
 		(unit 1)
@@
 			)
 		)
-		(property "Footprint" "SEBoard:RC0402N_YAG"
+		(property "Footprint" "000MCLib:RC0402N_YAG"
 			(at 185.42 118.11 0)
 			(effects
@@
 	)
 	(symbol
-		(lib_id "SEBoard:GRM155R60J106ME15D")
+		(lib_id "000MCLib:GRM155R60J106ME15D")
 		(at 242.57 63.5 270)
 		(unit 1)
@@
 			)
 		)
-		(property "Footprint" "SEBoard:CAPC1005X55N"
+		(property "Footprint" "000MCLib:CAPC1005X55N"
 			(at 146.38 72.39 0)
 			(effects
@@
 	)
 	(symbol
-		(lib_id "SEBoard:B140WS-7")
+		(lib_id "000MCLib:B140WS-7")
 		(at 207.01 125.73 270)
 		(unit 1)
@@
 			)
 		)
-		(property "Footprint" "SEBoard:SOD2513X120N"
+		(property "Footprint" "000MCLib:SOD2513X120N"
 			(at 113.36 138.43 0)
 			(effects
@@
 	)
 	(symbol
-		(lib_id "SEBoard:HD-EMB1104-SM-2")
+		(lib_id "000MCLib:HD-EMB1104-SM-2")
 		(at 222.25 118.11 0)
 		(unit 1)
@@
 			)
 		)
-		(property "Footprint" "SEBoard:PUI_HD-EMB1104-SM-2"
+		(property "Footprint" "000MCLib:PUI_HD-EMB1104-SM-2"
 			(at 222.25 118.11 0)
 			(effects
@@
 	)
 	(symbol
-		(lib_id "SEBoard:MMC3630KJ")
+		(lib_id "000MCLib:MMC3630KJ")
 		(at 74.93 53.34 0)
 		(unit 1)
@@
 			)
 		)
-		(property "Footprint" "SEBoard:BGA8C40P3X3_120X120X57"
+		(property "Footprint" "000MCLib:BGA8C40P3X3_120X120X57"
 			(at 99.06 148.26 0)
 			(effects
@@
 	)
 	(symbol
-		(lib_id "SEBoard:SML-P11VTT86R")
+		(lib_id "000MCLib:SML-P11VTT86R")
 		(at 45.72 114.3 90)
 		(unit 1)
@@
 			)
 		)
-		(property "Footprint" "SEBoard:SMLP11VTT86R"
+		(property "Footprint" "000MCLib:SMLP11VTT86R"
 			(at 139.37 101.6 0)
 			(effects
@@
 	)
 	(symbol
-		(lib_id "SEBoard:LIS2DH12TR")
+		(lib_id "000MCLib:LIS2DH12TR")
 		(at 208.28 53.34 0)
 		(unit 1)
@@
 			)
 		)
-		(property "Footprint" "SEBoard:LGA-12_STM"
+		(property "Footprint" "000MCLib:LGA-12_STM"
 			(at 177.8 46.99 0)
 			(effects
@@
 	)
 	(symbol
-		(lib_id "SEBoard:RC0402JR-072K2L")
+		(lib_id "000MCLib:RC0402JR-072K2L")
 		(at 45.72 128.27 90)
 		(unit 1)
@@
 			)
 		)
-		(property "Footprint" "SEBoard:RC0402N_YAG"
+		(property "Footprint" "000MCLib:RC0402N_YAG"
 			(at 45.72 134.62 0)
 			(effects
@@
 	)
 	(symbol
-		(lib_id "SEBoard:RC0402JR-072K2L")
+		(lib_id "000MCLib:RC0402JR-072K2L")
 		(at 111.76 133.35 270)
 		(unit 1)
@@
 			)
 		)
-		(property "Footprint" "SEBoard:RC0402N_YAG"
+		(property "Footprint" "000MCLib:RC0402N_YAG"
 			(at 111.76 127 0)
 			(effects
