File: 04_Hardware/PCBs/SEBoard/Interfaces.kicad_sch (KiCad schematic)
At the start: 63 parts, among them J12 67996-100HLF, J2 10-89-7121, Q1 BC847C,215, Q10 BC817-40,215, Q2 BC847C,215, Q3 BC847C,215, Q4 BC817-40,215, Q5 BC817-40,215, Q7 BC817-40,215, Q8 BC817-40,215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

Commit message: feat: Updated schematic
Connections:
- net AUDIO_EN: now also U5.C19 (PM_GPIO4); no longer U5.B20 (PM_GPIO3)
- net LCM_VCC_EN: now also U5.G19 (PM_GPIO8); no longer U5.C19 (PM_GPIO4)
- net NFC_VDD_EN: now also U5.B20 (PM_GPIO3); no longer U5.C27 (NFC_CLKREQ/GPIO_86)
- net at TP34.1: now also U5.C27 (NFC_CLKREQ/GPIO_86); no longer U5.G19 (PM_GPIO8)
Changed lines of the file:
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@@
 	(wire
 		(pts
+			(xy 80.01 140.97) (xy 63.5 140.97)
+		)
+		(stroke
+			(width 0)
+			(type default)
+		)
+	)
+	(wire
+		(pts
 			(xy 356.87 59.69) (xy 356.87 69.85)
 		)
@@
 	(wire
 		(pts
-			(xy 63.5 140.97) (xy 80.01 140.97)
-		)
-		(stroke
-			(width 0)
-			(type default)
-		)
-	)
-	(wire
-		(pts
 			(xy 251.46 213.36) (xy 257.81 213.36)
 		)
@@
 	(wire
 		(pts
-			(xy 80.01 137.16) (xy 63.5 137.16)
+			(xy 166.37 224.79) (xy 172.72 224.79)
 		)
 		(stroke
@@
 	(wire
 		(pts
-			(xy 166.37 224.79) (xy 172.72 224.79)
+			(xy 201.93 227.33) (xy 195.58 227.33)
 		)
 		(stroke
@@
 	(wire
 		(pts
-			(xy 201.93 227.33) (xy 195.58 227.33)
+			(xy 285.75 69.85) (xy 288.29 69.85)
 		)
 		(stroke
@@
 	(wire
 		(pts
-			(xy 285.75 69.85) (xy 288.29 69.85)
+			(xy 152.4 198.12) (xy 180.34 198.12)
 		)
 		(stroke
@@
 	(wire
 		(pts
-			(xy 80.01 144.78) (xy 63.5 144.78)
+			(xy 201.93 222.25) (xy 195.58 222.25)
 		)
 		(stroke
@@
 	(wire
 		(pts
-			(xy 152.4 198.12) (xy 180.34 198.12)
+			(xy 80.01 144.78) (xy 63.5 144.78)
 		)
 		(stroke
@@
 	(wire
 		(pts
-			(xy 201.93 222.25) (xy 195.58 222.25)
+			(xy 80.01 187.96) (xy 63.5 187.96)
 		)
 		(stroke
@@
 	(wire
 		(pts
-			(xy 85.09 215.9) (xy 63.5 215.9)
+			(xy 80.01 137.16) (xy 63.5 137.16)
 		)
 		(stroke
@@
 	(wire
 		(pts
-			(xy 289.56 105.41) (xy 289.56 115.57)
+			(xy 85.09 215.9) (xy 63.5 215.9)
 		)
 		(stroke
@@
 	(wire
 		(pts
-			(xy 372.11 67.31) (xy 372.11 69.85)
+			(xy 289.56 105.41) (xy 289.56 115.57)
 		)
 		(stroke
@@
 	(wire
 		(pts
-			(xy 270.51 213.36) (xy 270.51 223.52)
+			(xy 372.11 67.31) (xy 372.11 69.85)
 		)
 		(stroke
@@
 	(wire
 		(pts
-			(xy 201.93 229.87) (xy 195.58 229.87)
+			(xy 270.51 213.36) (xy 270.51 223.52)
 		)
 		(stroke
@@
 	(wire
 		(pts
-			(xy 80.01 187.96) (xy 63.5 187.96)
+			(xy 201.93 229.87) (xy 195.58 229.87)
 		)
 		(stroke
@@
 	(global_label "LCM_VCC_EN"
 		(shape output)
-		(at 80.01 140.97 0)
+		(at 80.01 144.78 0)
 		(fields_autoplaced yes)
 		(effects
@@
 		)
 		(property "Intersheetrefs" "${INTERSHEET_REFS}"
-			(at 94.788 140.97 0)
+			(at 94.788 144.78 0)
 			(effects
 				(font
@@
 	(global_label "AUDIO_EN"
 		(shape output)
-		(at 80.01 137.16 0)
+		(at 80.01 140.97 0)
 		(fields_autoplaced yes)
 		(effects
@@
 		)
 		(property "Intersheetrefs" "${INTERSHEET_REFS}"
-			(at 92.0667 137.16 0)
+			(at 92.0667 140.97 0)
 			(effects
 				(font
@@
 	)
 	(global_label "NFC_VDD_EN"
-		(shape input)
-		(at 80.01 187.96 0)
+		(shape output)
+		(at 80.01 137.16 0)
 		(fields_autoplaced yes)
 		(effects
@@
 		)
 		(property "Intersheetrefs" "${INTERSHEET_REFS}"
-			(at 94.7276 187.96 0)
+			(at 94.7276 137.16 0)
 			(effects
 				(font
@@
 	)
 	(symbol
+		(lib_id "000MCLib:TestPoint")
+		(at 80.01 187.96 270)
+		(unit 1)
+		(exclude_from_sim no)
+		(in_bom yes)
+		(on_board yes)
+		(dnp no)
+		(property "Reference" "TP34"
+			(at 84.328 187.96 90)
+			(effects
+				(font
+					(size 1.27 1.27)
+				)
+				(justify left)
+			)
+		)
+		(property "Value" "Sens_M"
+			(at 80.264 188.976 90)
+			(effects
+				(font
+					(size 0.635 0.635)
+				)
+				(hide yes)
+			)
+		)
+		(property "Footprint" "TestPoint:TestPoint_Pad_D1.0mm"
+			(at 80.01 193.04 0)
+			(effects
+				(font
+					(size 1.27 1.27)
+				)
+				(hide yes)
+			)
+		)
+		(property "Datasheet" "~"
+			(at 80.01 193.04 0)
+			(effects
+				(font
+					(size 1.27 1.27)
+				)
+				(hide yes)
+			)
+		)
+		(property "Description" "test point"
+			(at 80.01 187.96 0)
+			(effects
+				(font
+					(size 1.27 1.27)
+				)
+				(hide yes)
+			)
+		)
+		(pin "1"
+		)
+		(instances
+			(project "SEBoard"
+				(path "/38605b01-fdd9-41de-8a8b-501279ee3e8a/b1e534e0-0f7b-45a3-a276-524cb0179f18"
+					(reference "TP34")
+					(unit 1)
+				)
+			)
+		)
+	)
+	(symbol
 		(lib_id "power:VDD")
 		(at 330.2 38.1 0)
@@
 					(unit 1)
 				)
-			)
-		)
-	)
-	(symbol
-		(lib_id "000MCLib:TestPoint")
-		(at 80.01 144.78 270)
-		(unit 1)
-		(exclude_from_sim no)
-		(in_bom yes)
-		(on_board yes)
-		(dnp no)
-		(property "Reference" "TP34"
-			(at 84.328 144.78 90)
-			(effects
-				(font
-					(size 1.27 1.27)
-				)
-				(justify left)
-			)
-		)
-		(property "Value" "Sens_M"
-			(at 80.264 145.796 90)
-			(effects
-				(font
-					(size 0.635 0.635)
-				)
-				(hide yes)
-			)
-		)
-		(property "Footprint" "TestPoint:TestPoint_Pad_D1.0mm"
-			(at 80.01 149.86 0)
-			(effects
-				(font
-					(size 1.27 1.27)
-				)
-				(hide yes)
-			)
-		)
-		(property "Datasheet" "~"
-			(at 80.01 149.86 0)
-			(effects
-				(font
-					(size 1.27 1.27)
-				)
-				(hide yes)
-			)
-		)
-		(property "Description" "test point"
-			(at 80.01 144.78 0)
-			(effects
-				(font
-					(size 1.27 1.27)
-				)
-				(hide yes)
-			)
-		)
-		(pin "1"
-		)
-		(instances
-			(project "SEBoard"
-				(path "/38605b01-fdd9-41de-8a8b-501279ee3e8a/b1e534e0-0f7b-45a3-a276-524cb0179f18"
-					(reference "TP34")
-					(unit 1)
-				)
