File: 04_Hardware/PCBs/SEBoard/SEBoard.kicad_pcb (KiCad board)
At the start: 6 copper layers, 80 x 140.6 mm, 442 parts, among them IC1 PN7220, IC2 ST4SI2M0020TPIFW, IC3 PCA9306DCTT, IC4 TXS0102DCUR, IC5 LM74700QDBVRQ1, J1 PJ-059A, J10 67996-100HLF, J12 67996-100HLF, J13 YXT-BB10-30S-02, J14 FH12S-30S-0.5SH_55_, J15 FH12-8S-0.5SH_55_, J16 SIM8066-6-1-14-01-A, J17 MEM2067-02-180-00-A, J18 636101112001, J19 636101112001, J2 10-89-7121, J20 636101112001, J21 636101112001, J22 53047-0210, J3 53047-0310, J4 67996-100HLF, J5 USB4080-03-A, J6 22-28-4034, J7 BM02B-ACHSS-GAN-TF, J9 22-28-4034, Q1 BC847C,215, Q10 BC817-40,215, Q11 BC847C,215, Q12 BC847C,215, Q13 AO3400A, Q2 BC847C,215, Q3 BC847C,215, Q4 BC817-40,215, Q5 BC817-40,215, Q7 BC817-40,215, Q8 BC817-40,215, Q9 BC817-40,215, U100 PAM8302AASCR, U2 RT8279GSP, U3 AP7335-WG-7, U4 AP7343DQ-11W5-7, U5 SE250B4, U6 LIS2DH12TR, U7 MMC3630KJ, U8 AP61100Z6-7, U9 AP5724WG-7, Y1 27.120MHz

Commit message: fix: Solved DRCs but not all
Parts:
- moved D1 0.43 mm to (132.4, 156.8)
- moved J1 0.30 mm to (133.1, 160.2)
- moved C1 0.12 mm to (123.5, 170.1)
Routing:
- net ACCL_INT: track 39.6 -> 41.3 mm
- net VUSB_BUS: track 45.1 -> 46.3 mm
- net Net-(U5Power-VREG_S4A_2P04): track 9.60 -> 8.51 mm
- net /SIM_SD/USIM1_VDD: track 45.5 -> 44.8 mm
- net /Interfaces/GPIO_IN3: track 21.8 -> 22.5 mm
- net GND: track 70.9 -> 71.5 mm, vias 409 -> 408
- net /Audio/MIC_BIAS1: track 21.8 -> 22.3 mm
